File: pcb/USB_Analog_Controller.brd (EAGLE design)
At the start: 50 x 36 mm, 24 parts, among them J1 POWER, Q1 AO3400, Q2 AO3400, U1 PICO-MINI-02, U2 AP2112K, X1 PROG, X2 LED1, X3 LED2, X5 BOOT, X6 RESET

Commit message: Revision 2023-08-04 Switch power connector Add PDF file Cleanup old PCB files
Parts:
- F1, F2: value 3A -> JK-SMD300L-16
- J1: device M2M-Connectors:TERMINAL-5.08-2P -> M2M-Connectors:TERMINAL-2.54-2P
- U1: value PICO-MINI-02 -> ESP32-PICO-MINI-02
- X2: value LED1 -> SS-52100-001
- X3: value LED2 -> SS-52100-001
Connections:
- net GND: now also J1.2; no longer J1.P$2
- net VIN: now also J1.1; no longer J1.P$1
Other:
- board text added: "2023-08-04"
- board text removed: "2023-07-27"
Changed lines of the file:
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@@
 <setting verticaltext="up"/>
 </settings>
-<grid distance="0.5" unitdist="mm" unit="mm" style="lines" multiple="1" display="no" altdistance="5" altunitdist="mil" altunit="mil"/>
+<grid distance="0.5" unitdist="mm" unit="mm" style="lines" multiple="1" display="yes" altdistance="0.1" altunitdist="mm" altunit="mm"/>
 <layers>
 <layer number="1" name="Top" color="4" fill="1" visible="yes" active="yes"/>
@@
 <text x="48.5" y="6" size="1.27" layer="21" rot="R90">USB Analog
 Controller</text>
-<text x="48.5" y="20" size="1.016" layer="21" rot="R90">2023-07-27</text>
-<text x="44" y="12.5" size="1.27" layer="21" rot="R90">GND</text>
-<text x="44" y="7.5" size="1.27" layer="21" rot="R90">5V</text>
+<text x="48.5" y="20" size="1.016" layer="21" rot="R90">2023-08-04</text>
+<text x="40.5" y="12.5" size="1.27" layer="21">GND</text>
+<text x="40.5" y="9.5" size="1.27" layer="21">5V</text>
 <dimension x1="18" y1="18" x2="0" y2="18" x3="9" y3="-4.5" textsize="1.778" layer="47"/>
 <dimension x1="45" y1="18" x2="0" y2="18" x3="22.5" y3="-8.5" textsize="1.778" layer="47"/>
@@
 <attribute name="VALUE" x="18.5" y="14.905" size="1.016" layer="27" rot="R180" align="bottom-center"/>
 </element>
-<element name="U1" library="M2M-Modules" package="ESP32-PICO-MINI-02" value="PICO-MINI-02" x="34" y="24.5" smashed="yes"/>
+<element name="U1" library="M2M-Modules" package="ESP32-PICO-MINI-02" value="ESP32-PICO-MINI-02" x="34" y="24.5" smashed="yes"/>
 <element name="X1" library="M2M-Connectors" package="FTDI232-1X06" value="PROG" x="38.5" y="3.5" smashed="yes" rot="R90">
 <attribute name="NAME" x="29.9275" y="2.23" size="1.016" layer="26" rot="R90"/>
@@
 <attribute name="VALUE" x="30.73" y="0.975" size="1.016" layer="21"/>
 </element>
-<element name="X2" library="M2M-Connectors" package="USB-A-SS-52100-001" value="LED1" x="10" y="27" smashed="yes" rot="R90">
+<element name="X2" library="M2M-Connectors" package="USB-A-SS-52100-001" value="SS-52100-001" x="10" y="27" smashed="yes" rot="R90">
 <attribute name="NAME" x="8" y="19.5" size="1.27" layer="25" rot="R180"/>
 <attribute name="NAME" x="6" y="27" size="1.27" layer="51" rot="R90" align="center"/>
 <attribute name="VALUE" x="8.1" y="35.7" size="1.27" layer="27" rot="R180"/>
 </element>
-<element name="X3" library="M2M-Connectors" package="USB-A-SS-52100-001" value="LED2" x="10" y="9" smashed="yes" rot="R90">
+<element name="X3" library="M2M-Connectors" package="USB-A-SS-52100-001" value="SS-52100-001" x="10" y="9" smashed="yes" rot="R90">
 <attribute name="NAME" x="8" y="1.5" size="1.27" layer="25" rot="R180"/>
 <attribute name="NAME" x="6" y="9" size="1.27" layer="51" rot="R90" align="center"/>
@@
 </element>
 <element name="X5" library="M2M-Connectors" package="1X02-2.54" value="BOOT" x="25.5" y="3.5" smashed="yes">
+<attribute name="NAME" x="24.865" y="2.865" size="0.8128" layer="51"/>
 <attribute name="NAME" x="24.23" y="5.0875" size="1.016" layer="25"/>
 <attribute name="NAME" x="24.611" y="2.865" size="1.27" layer="48"/>
-<attribute name="NAME" x="24.865" y="2.865" size="0.8128" layer="51"/>
 <attribute name="VALUE" x="24.23" y="0.96" size="1.016" layer="21"/>
 </element>
 <element name="X6" library="M2M-Connectors" package="1X02-2.54" value="RESET" x="19" y="3.5" smashed="yes">
+<attribute name="NAME" x="18.865" y="2.365" size="0.8128" layer="51"/>
 <attribute name="NAME" x="17.73" y="5.0875" size="1.016" layer="25"/>
 <attribute name="NAME" x="18.111" y="2.865" size="1.27" layer="48"/>
-<attribute name="NAME" x="18.865" y="2.365" size="0.8128" layer="51"/>
 <attribute name="VALUE" x="17.73" y="0.96" size="1.016" layer="21"/>
 </element>
-<element name="J1" library="M2M-Connectors" package="TERMINAL-5.08-2P" value="POWER" x="37" y="11.5" smashed="yes" rot="R90"/>
+<element name="J1" library="M2M-Connectors" package="TERMINAL-2.54-2P" value="POWER" x="37" y="11.5" smashed="yes" rot="R90"/>
 <element name="U2" library="M2M-IC" package="SOT23-5" value="AP2112K" x="27.5" y="13" smashed="yes">
 <attribute name="NAME" x="27.495" y="14.805" size="1.016" layer="25" align="bottom-center"/>
@@
 <attribute name="VALUE" x="25.5" y="4.595" size="1.016" layer="27" align="bottom-center"/>
 </element>
-<element name="F1" library="M2M-Fuse" package="JK-SMD300" value="3A" x="6" y="27" smashed="yes" rot="MR180">
+<element name="F1" library="M2M-Fuse" package="JK-SMD300" value="JK-SMD300L-16" x="6" y="27" smashed="yes" rot="MR180">
 <attribute name="NAME" x="1" y="23.5" size="1.016" layer="26" rot="MR180"/>
 <attribute name="NAME" x="6" y="27" size="1.016" layer="48" rot="MR180" align="center"/>
 <attribute name="VALUE" x="1" y="31.5" size="1.016" layer="28" rot="MR180"/>
 </element>
-<element name="F2" library="M2M-Fuse" package="JK-SMD300" value="3A" x="6" y="9" smashed="yes" rot="MR180">
+<element name="F2" library="M2M-Fuse" package="JK-SMD300" value="JK-SMD300L-16" x="6" y="9" smashed="yes" rot="MR180">
 <attribute name="NAME" x="1" y="5.5" size="1.016" layer="26" rot="MR180"/>
 <attribute name="NAME" x="6" y="9" size="1.016" layer="48" rot="MR180" align="center"/>
@@
 <contactref element="Q1" pad="2"/>
 <contactref element="Q2" pad="2"/>
-<contactref element="J1" pad="P$2"/>
+<contactref element="J1" pad="2"/>
 <polygon width="0.1524" layer="1">
 <vertex x="0" y="36"/>
@@
 <signal name="VIN">
 <contactref element="U2" pad="1"/>
-<contactref element="J1" pad="P$1"/>
+<contactref element="J1" pad="1"/>
 <contactref element="C3" pad="1"/>
 <contactref element="U2" pad="3"/>
 <contactref element="C2" pad="1"/>
-<wire x1="30.5" y1="10.35" x2="29.5" y2="10.35" width="1.016" layer="1"/>
 <via x="30" y="11.5" extent="1-16" drill="0.8"/>
-<wire x1="30" y1="11.5" x2="30.5" y2="11" width="1.016" layer="1"/>
-<wire x1="30.5" y1="11" x2="30.5" y2="10.35" width="1.016" layer="1"/>
 <wire x1="28.45" y1="11.7" x2="28.45" y2="10.6" width="0.4064" layer="1"/>
 <wire x1="28.45" y1="10.6" x2="27.85" y2="10" width="0.4064" layer="1"/>
@@
 <wire x1="7.2" y1="5.3" x2="10.7" y2="5.3" width="1.016" layer="16"/>
 <wire x1="3.5" y1="9" x2="7.2" y2="5.3" width="1.016" layer="16"/>
-<wire x1="35.61" y1="10.35" x2="37" y2="8.96" width="1.016" layer="1"/>
-<wire x1="30.5" y1="10.35" x2="35.61" y2="10.35" width="1.016" layer="1"/>
+<wire x1="37" y1="10.23" x2="31.27" y2="10.23" width="1.016" layer="1"/>
+<wire x1="31.15" y1="10.35" x2="30" y2="11.5" width="1.016" layer="1"/>
+<wire x1="29.5" y1="10.35" x2="31.15" y2="10.35" width="1.016" layer="1"/>
+<wire x1="31.15" y1="10.35" x2="31.27" y2="10.23" width="1.016" layer="1"/>
 </signal>
 <signal name="N$5">
