File: pcb/USB_Analog_Controller 24V.brd (EAGLE design)
At the start: 50 x 36 mm, 29 parts, among them J1 POWER, Q1 AO3400, Q2 AO3400, U1 ESP32-PICO-MINI-02, X1 PROG, X2 L1, X3 L2, X5 BOOT, X6 RESET

Commit message: Change connector on24V PCB Cosmetic fixes on 24V PCB
Parts:
- added U$4: (no value), M2M-Frames:OSHW-5MM-TPLACE
- added U$5: (no value), M2M-Frames:BERGDAHL-20MM-TPLACE
- J1: device M2M-Connectors:TERMINAL-2.54-2P -> M2M-Connectors:TERMINAL-5.08-2P
- moved J1 1.80 mm to (38.5, 10.5)
Connections:
- net GND: now also J1.P$2; no longer J1.2
- net VIN: now also J1.P$1; no longer J1.1
Routing:
- net VIN: track 47.6 -> 63.2 mm
- net IO0: track 34.6 -> 37.0 mm
- net VCC: track 36.7 -> 35.3 mm
Other:
- board text added: "2023-08-14"
- board text added: "Analog LED Controller 5-24V"
- board text removed: "2023-08-09"
- board text removed: "USB Analog Controller 5-24V"
Changed lines of the file:
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@@
 <drawing>
 <settings>
-<setting alwaysvectorfont="no"/>
+<setting alwaysvectorfont="yes"/>
 <setting verticaltext="up"/>
 </settings>
@@
 <wire x1="23.5" y1="36" x2="2" y2="36" width="0" layer="20"/>
 <wire x1="2" y1="36" x2="0" y2="34" width="0" layer="20" curve="90"/>
-<text x="48.5" y="6" size="1.27" layer="21" rot="R90">USB Analog
+<text x="2" y="1.5" size="1.27" layer="21">Analog LED
 Controller 5-24V</text>
-<text x="48.5" y="20" size="1.016" layer="21" rot="R90">2023-08-09</text>
-<text x="40.5" y="12.5" size="1.27" layer="21">GND</text>
-<text x="40.5" y="9.5" size="1.27" layer="21">5-24V</text>
+<text x="49" y="3" size="1.016" layer="21" rot="R90">2023-08-14</text>
+<text x="46" y="11.5" size="1.27" layer="21" rot="R90">GND</text>
+<text x="46" y="5.5" size="1.27" layer="21" rot="R90">5-24V</text>
 <dimension x1="18" y1="18" x2="0" y2="18" x3="9" y3="-4.5" textsize="1.778" layer="47"/>
 <dimension x1="45" y1="18" x2="0" y2="18" x3="22.5" y3="-8.5" textsize="1.778" layer="47"/>
@@
 </element>
 <element name="X5" library="M2M-Connectors" package="1X02-2.54" value="BOOT" x="25.5" y="3.5" smashed="yes">
+<attribute name="NAME" x="24.23" y="5.0875" size="1.016" layer="25"/>
 <attribute name="NAME" x="24.611" y="2.865" size="1.27" layer="48"/>
 <attribute name="NAME" x="24.865" y="2.865" size="0.8128" layer="51"/>
-<attribute name="NAME" x="24.23" y="5.0875" size="1.016" layer="25"/>
 <attribute name="VALUE" x="24.23" y="0.96" size="1.016" layer="21"/>
 </element>
 <element name="X6" library="M2M-Connectors" package="1X02-2.54" value="RESET" x="19" y="3.5" smashed="yes">
+<attribute name="NAME" x="17.73" y="5.0875" size="1.016" layer="25"/>
 <attribute name="NAME" x="18.111" y="2.865" size="1.27" layer="48"/>
 <attribute name="NAME" x="18.865" y="2.365" size="0.8128" layer="51"/>
-<attribute name="NAME" x="17.73" y="5.0875" size="1.016" layer="25"/>
 <attribute name="VALUE" x="17.73" y="0.96" size="1.016" layer="21"/>
 </element>
-<element name="J1" library="M2M-Connectors" package="TERMINAL-2.54-2P" value="POWER" x="37" y="11.5" smashed="yes" rot="R90"/>
+<element name="J1" library="M2M-Connectors" package="TERMINAL-5.08-2P" value="POWER" x="38.5" y="10.5" smashed="yes" rot="R90"/>
 <element name="R3" library="M2M-Passives" package="R0603" value="10K" x="18.5" y="24.5" smashed="yes" rot="R90">
 <attribute name="NAME" x="17.5475" y="24.5" size="1.016" layer="25" rot="R90" align="bottom-center"/>
@@
 <attribute name="VALUE" x="9.5" y="16.5" size="1.27" layer="27" align="bottom-right"/>
 </element>
+<element name="U$4" library="M2M-Frames" package="OSHW-5MM-TPLACE" value="" x="46" y="24.5" smashed="yes"/>
+<element name="U$5" library="M2M-Frames" package="BERGDAHL-20MM-TPLACE" value="" x="5" y="30.5" smashed="yes"/>
 </elements>
 <signals>
@@
 <wire x1="28.1" y1="26.9" x2="25.75" y2="26.9" width="0.6096" layer="1"/>
 <wire x1="25.75" y1="26.9" x2="25.5" y2="26.65" width="0.6096" layer="1"/>
-<wire x1="20.5" y1="12.35" x2="20.35" y2="12.5" width="0.6096" layer="1"/>
-<wire x1="20.35" y1="12.5" x2="19.5" y2="12.5" width="0.6096" layer="1"/>
-<via x="19.5" y="12.5" extent="1-16" drill="0.35"/>
-<wire x1="19.5" y1="12.5" x2="20.5" y2="13.5" width="0.6096" layer="16"/>
-<wire x1="20.5" y1="23" x2="20.5" y2="13.5" width="0.6096" layer="16"/>
+<wire x1="20.5" y1="12.35" x2="20.5" y2="13" width="0.6096" layer="1"/>
+<via x="20.5" y="13" extent="1-16" drill="0.35"/>
+<wire x1="20.5" y1="23" x2="20.5" y2="13" width="0.6096" layer="16"/>
 <wire x1="20.5" y1="23" x2="24" y2="26.5" width="0.6096" layer="16"/>
 <via x="24" y="26.5" extent="1-16" drill="0.35"/>
@@
 <contactref element="Q1" pad="2"/>
 <contactref element="Q2" pad="2"/>
-<contactref element="J1" pad="2"/>
+<contactref element="J1" pad="P$2"/>
 <polygon width="0.1524" layer="1" rank="5">
 <vertex x="0" y="36"/>
@@
 <contactref element="X5" pad="1"/>
 <wire x1="38" y1="19" x2="38" y2="19.6" width="0.254" layer="1"/>
-<wire x1="39.5" y1="17.5" x2="39.5" y2="7.5" width="0.254" layer="1"/>
-<wire x1="39.5" y1="17.5" x2="38" y2="19" width="0.254" layer="1"/>
+<wire x1="41" y1="16" x2="38" y2="19" width="0.254" layer="1"/>
 <contactref element="R5" pad="1"/>
-<wire x1="39.5" y1="7.5" x2="36" y2="4" width="0.254" layer="1"/>
-<wire x1="36" y1="4" x2="36" y2="3" width="0.254" layer="1"/>
+<wire x1="36" y1="3" x2="36" y2="4" width="0.254" layer="1"/>
 <wire x1="36" y1="3" x2="35" y2="2" width="0.254" layer="1"/>
 <wire x1="35" y1="2" x2="27" y2="2" width="0.254" layer="1"/>
@@
 <wire x1="22" y1="5.65" x2="24.15" y2="3.5" width="0.254" layer="1"/>
 <wire x1="24.15" y1="3.5" x2="25.5" y2="3.5" width="0.254" layer="1"/>
+<wire x1="36" y1="4" x2="37" y2="5" width="0.254" layer="1"/>
+<wire x1="39" y1="5" x2="41" y2="7" width="0.254" layer="1"/>
+<wire x1="37" y1="5" x2="39" y2="5" width="0.254" layer="1"/>
+<wire x1="41" y1="7" x2="41" y2="16" width="0.254" layer="1"/>
 </signal>
 <signal name="EN">
@@
 <contactref element="X2" pad="2"/>
 <contactref element="X2" pad="3"/>
-<wire x1="15.5" y1="22.9" x2="12.4" y2="19.8" width="1.016" layer="1"/>
-<wire x1="12.4" y1="19.8" x2="6.5" y2="19.8" width="1.016" layer="1"/>
-<wire x1="6.5" y1="19.8" x2="3.6" y2="22.7" width="1.016" layer="1"/>
-<wire x1="3.6" y1="22.7" x2="3.6" y2="24.5" width="1.016" layer="1"/>
+<wire x1="3.6" y1="24.5" x2="3.6" y2="22.7" width="1.5" layer="1"/>
+<wire x1="3.6" y1="22.7" x2="6.5" y2="19.8" width="1.5" layer="1"/>
+<wire x1="6.5" y1="19.8" x2="12.4" y2="19.8" width="1.5" layer="1"/>
+<wire x1="12.4" y1="19.8" x2="15.5" y2="22.9" width="1.5" layer="1"/>
 </signal>
 <signal name="N$2">
@@
 <contactref element="X3" pad="3"/>
 <contactref element="X3" pad="2"/>
-<wire x1="6.5" y1="6.8" x2="3.6" y2="9.7" width="1.016" layer="1"/>
-<wire x1="3.6" y1="9.7" x2="3.6" y2="11.5" width="1.016" layer="1"/>
-<wire x1="15.5" y1="8.9" x2="13.4" y2="6.8" width="1.016" layer="1"/>
-<wire x1="13.4" y1="6.8" x2="6.5" y2="6.8" width="1.016" layer="1"/>
+<wire x1="5.4906" y1="7.7702" x2="5.5298" y2="7.7702" width="1.5" layer="1"/>
+<wire x1="5.5298" y1="7.7702" x2="6.5" y2="6.8" width="1.5" layer="1"/>
+<wire x1="3.6" y1="11.5" x2="3.6" y2="9.6608" width="1.5" layer="1"/>
+<wire x1="3.6" y1="9.6608" x2="5.4906" y2="7.7702" width="1.5" layer="1"/>
+<wire x1="6.5" y1="6.8" x2="13.4" y2="6.8" width="1.5" layer="1"/>
+<wire x1="13.4" y1="6.8" x2="15.5" y2="8.9" width="1.5" layer="1"/>
 </signal>
 <signal name="N$3">
@@
 </signal>
 <signal name="VIN">
-<contactref element="J1" pad="1"/>
+<contactref element="J1" pad="P$1"/>
 <contactref element="F1" pad="A"/>
 <contactref element="F2" pad="A"/>
@@
 <contactref element="U$3" pad="4"/>
 <polygon width="0.1524" layer="1">
-<vertex x="38.5" y="11.5"/>
+<vertex x="40.5" y="11.5"/>
 <vertex x="34.8" y="11.5"/>
 <vertex x="32.5" y="9.2"/>
@@
 <vertex x="31.4" y="5.5"/>
 <vertex x="32.3" y="5.5"/>
-<vertex x="35.6" y="8.8"/>
-<vertex x="38.3" y="8.8"/>
-<vertex x="38.5" y="9"/>
+<vertex x="33.6" y="6.8"/>
+<vertex x="39.3" y="6.8"/>
+<vertex x="40.5" y="8"/>
 </polygon>
-<wire x1="35.23" y1="10.23" x2="31" y2="6" width="1.016" layer="16"/>
-<wire x1="35.23" y1="10.23" x2="37" y2="10.23" width="1.016" layer="16"/>
-<wire x1="7" y1="10" x2="7" y2="14" width="1.016" layer="16"/>
-<wire x1="14" y1="21" x2="14" y2="21.3" width="1.016" layer="16"/>
-<wire x1="7" y1="10" x2="9.7" y2="7.3" width="1.016" layer="16"/>
-<wire x1="7" y1="14" x2="14" y2="21" width="1.016" layer="16"/>
-<wire x1="9.7" y1="7.3" x2="14" y2="7.3" width="1.016" layer="16"/>
-<wire x1="15.3" y1="6" x2="14" y2="7.3" width="1.016" layer="16"/>
-<wire x1="31" y1="6" x2="15.3" y2="6" width="1.016" layer="16"/>
+<wire x1="38.5" y1="7.96" x2="36.04" y2="5.5" width="1.5" layer="16"/>
+<wire x1="15.8" y1="5.5" x2="14" y2="7.3" width="1.5" layer="16"/>
+<wire x1="36.04" y1="5.5" x2="15.8" y2="5.5" width="1.5" layer="16"/>
+<wire x1="14" y1="21.3" x2="9.7" y2="17" width="1.5" layer="16"/>
+<wire x1="4.5" y1="17" x2="1.5" y2="14" width="1.5" layer="16"/>
+<wire x1="1.5" y1="14" x2="1.5" y2="7.5" width="1.5" layer="16"/>
+<wire x1="11.2" y1="4.5" x2="14" y2="7.3" width="1.5" layer="16"/>
+<wire x1="9.7" y1="17" x2="4.5" y2="17" width="1.5" layer="16"/>
+<wire x1="1.5" y1="7.5" x2="4.5" y2="4.5" width="1.5" layer="16"/>
+<wire x1="4.5" y1="4.5" x2="11.2" y2="4.5" width="1.5" layer="16"/>
 </signal>
 <signal name="N$5">
 <contactref element="F1" pad="B"/>
 <contactref element="X2" pad="1"/>
-<wire x1="14" y1="28.7" x2="9.8" y2="24.5" width="1.016" layer="16"/>
-<wire x1="9.8" y1="24.5" x2="9.5" y2="24.5" width="1.016" layer="16"/>
+<wire x1="14" y1="28.7" x2="9.8" y2="24.5" width="1.5" layer="16"/>
+<wire x1="9.8" y1="24.5" x2="9.5" y2="24.5" width="1.5" layer="16"/>
 </signal>
 <signal name="N$6">
 <contactref element="F2" pad="B"/>
 <contactref element="X3" pad="1"/>
-<wire x1="14" y1="14.7" x2="10.8" y2="11.5" width="1.016" layer="16"/>
-<wire x1="10.8" y1="11.5" x2="9.5" y2="11.5" width="1.016" layer="16"/>
+<wire x1="14" y1="14.7" x2="10.8" y2="11.5" width="1.5" layer="16"/>
+<wire x1="10.8" y1="11.5" x2="9.5" y2="11.5" width="1.5" layer="16"/>
 </signal>
 <signal name="N$7">
@@
 <wire x1="26.5" y1="7.85" x2="26.5" y2="9" width="0.254" layer="1"/>
 <wire x1="26.5" y1="9" x2="26.575" y2="9.075" width="0.254" layer="1"/>
-<wire x1="26.5" y1="7.85" x2="26.7" y2="8.05" width="0.254" layer="1"/>
 <wire x1="26.5" y1="9.15" x2="27.35" y2="9.15" width="0.254" layer="1"/>
 <wire x1="27.35" y1="9.15" x2="27.5" y2="9" width="0.254" layer="1"/>
