File: pcb/USB_Analog_Controller 24V.sch (EAGLE design)
At the start: 27 parts, among them J1 POWER, Q1 AO3400, Q2 AO3400, U1 ESP32-PICO-MINI-02, X1 PROG, X2 L1, X3 L2, X5 BOOT, X6 RESET

Commit message: Change connector on24V PCB Cosmetic fixes on 24V PCB
Parts:
- J1: device M2M-Connectors:TERMINAL-1X02-2.54P -> M2M-Connectors:TERMINAL-1X02-5.08
Changed lines of the file:
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@@
 <part name="GND10" library="M2M-Power" deviceset="GND" device=""/>
 <part name="SUPPLY6" library="M2M-Power" deviceset="VCC" device=""/>
-<part name="J1" library="M2M-Connectors" deviceset="TERMINAL-1X02-2.54" device="P" value="POWER"/>
+<part name="J1" library="M2M-Connectors" deviceset="TERMINAL-1X02-5.08" device="" value="POWER"/>
 <part name="SUPPLY2" library="M2M-Power" deviceset="VIN" device=""/>
 <part name="SUPPLY3" library="M2M-Power" deviceset="VIN" device=""/>
